File: assets/project/project.kicad_pcb (KiCad board)
At the start: 2 copper layers, 102.9 x 71.1 mm, 17 parts, among them J1 Micro SD, J2 EPD, J3 RTC, J4 Battery In, SW1 SW_SPDT, U1 Reset

Commit message: kicad
Parts:
- removed SW1: SW_SPDT, Button_Switch_THT:SW_Slide-03_Wuerth-WS-SLTV_10x2.5x6.4_P2.54mm
- added GND: GND, Connector_Pin:Pin_D1.3mm_L10.0mm_W3.5mm_Flat, F.Cu at (200.7, 94.2)
- added VIN: VIN, Connector_Pin:Pin_D1.3mm_L10.0mm_W3.5mm_Flat, F.Cu at (200.7, 99.0)
- added VOUT: VOUT, Connector_Pin:Pin_D1.3mm_L10.0mm_W3.5mm_Flat, F.Cu at (200.7, 103.7)
- C1 (0.1uF): renamed from C1; value C_US -> 0.1uF
- C2 (0.1uF): renamed from C2; value C_US -> 0.1uF
- R1 (1MΩ): renamed from R1; value R -> R (1M)
- R2 (1MΩ): renamed from R2; value R -> R (1M)
- U1: footprint Button_Switch_THT:SW_Push_2P1T_Toggle_CK_PVA1xxH1xxxxxxV2 -> Button_Switch_THT:SW_PUSH_6mm
- moved J4 3.94 mm to (195.7, 118.6)
Connections:
- A1 pad 30: Net-(A1-VIN) -> +4V
- R2 (1MΩ) pad 1: Net-(A1-VIN) -> +4V
Routing:
- net +4V: track 28.5 -> 140.7 mm, vias 0 -> 2
- net Net-(A1-VIN): track 94.0 -> 0.00 mm, vias 2 -> 0
- net Net-(A1-3V3): track 282.9 -> 279.1 mm, vias 4 -> 3
- net Net-(A1-D5): track 43.0 -> 40.7 mm
- net Net-(A1-D8): track 30.5 -> 28.2 mm
- net Net-(A1-D9): track 31.8 -> 29.9 mm
- net Net-(A1-D4): track 43.0 -> 41.1 mm
- net Net-(A1-D10/CS): track 33.0 -> 31.5 mm
- net Net-(A1-D3): track 43.0 -> 41.5 mm
Other:
- board text added: "-"
